File: docs/eagle/Led_display.sch (EAGLE design)
At the start: 42 parts, among them Q1 16 Mhz, U1 328P, U2 V_REG_317DPACK

Commit message: version 1.0
Parts:
- added C6: 100n, capacitor-wima:C2,5-3
Connections:
- net N$14: now also R12.1, U1.PB3(MOSI/OC2); no longer R14.1, U1.PD0(RXD)
- net N$15: now also U1.PB4(MISO); no longer U1.PD1(TXD)
- net N$16: now also R14.1, U1.PB5(SCK); no longer R12.1, U1.PD2(INT0)
- net N$29: now also R12.2; no longer R14.2
- net N$3: now also C6.2
- net N$31: now also R14.2; no longer R12.2
- net N$4: now also C6.1, U1.AVCC
- net N$7: no longer U1.PB3(MOSI/OC2)
- net N$8: now also R4.S
- net N$9: now also U1.PD2(INT0); no longer R4.S
Other:
- moved on the sheet: LED5, LED6, LED7, R12, R13, R14

Commit message: updating docs
Parts:
- added R19: 10K, eagle-ltspice:RR0402
- R10, R12, R13, R14, R15, R17, R18, R3, R5, R6, R8: value 120 -> 200
- R11, R16, R9: value (none) -> 200
- R4: value (none) -> POT
- S1: value MOMENTARY-SWITCH-SPST-PTH-6.0MM -> Push Button
- U2: value V_REG_317DPACK -> LM317
Connections:
- removed net N$4: C3.1, C6.1, R1.2, R4.E, U1.AVCC, U1.VCC, U2.OUT
- new net N$40: R19.2, U1.PC6(/RESET)
- new net N$41: C3.1, C6.1, R1.2, R19.1, R4.E, U1.AVCC, U1.VCC, U2.OUT

Commit message: adjusting schematic
Connections:
- removed net N$41 (its old number): C3.1, C6.1, R1.2, R19.1, R4.E, U1.AVCC, U1.VCC, U2.OUT
- removed net N$6: C4.2, R1.1, R2.2, U2.ADJ
- new net GND: C1.2, C2.2, C3.2, C4.2, C6.2, LED1.C, LED10.C, LED11.C, LED12.C, LED13.C, LED14.C, LED15.C, LED2.C, LED3.C, LED4.C, LED5.C, LED6.C, LED7.C, LED8.C, LED9.C, R2.1, R4.A, U1.GND@1
- new net N$4: R1.1, R2.2, U2.ADJ
- new net VCC: R19.1, R4.E
- net N$3: now also C3.1, C6.1, R1.2, U1.AVCC, U1.VCC, U2.OUT; no longer C1.2, C2.2, C3.2, C6.2, LED1.C, LED10.C, LED11.C, LED12.C, LED13.C, LED14.C, LED15.C, LED2.C, LED3.C, LED4.C, LED5.C, LED6.C, LED7.C, LED8.C, LED9.C, R2.1, R4.A, U1.GND@1
Other:
- moved on the sheet: C1, C6, R4
